Commit message: Ignoring urdf

File: urdf/fish.urdf.xacro (robot description, xacro)
@@ -22,6 +22,8 @@
     <collision>
       <geometry>
-        <mesh filename="file://$(find fish)/meshes/${model_name}" scale="${mesh_scale}" />
+        <box size="0.726 0.206 0.106"/>
+        <!--<mesh filename="file://$(find fish)/meshes/${model_name}" scale="${mesh_scale}" />-->
       </geometry>
+      <origin rpy="0.0 0.0 0.0" xyz="0.0 0.0 0.0" />
     </collision>
     <inertial>
@@ -46,6 +48,8 @@
     <collision>
       <geometry>
-        <mesh filename="file://$(find fish)/meshes/Tail.STL" scale="${mesh_scale}" />
+        <box size="0.272 0.210 0.0101"/>
+        <!--<mesh filename="file://$(find fish)/meshes/Tail.STL" scale="${mesh_scale}" />-->
       </geometry>
+      <origin rpy="0.0 0.0 0.0" xyz="0.14147 0.0 0.0"/>
     </collision>
     <inertial>

Commit message: Common commit

File: urdf/fish.urdf.xacro (robot description, xacro)
@@ -3,6 +3,6 @@
   <xacro:property name="mesh_scale" value="0.001 0.001 0.001" />
   <xacro:property name="body_center_gravity" value="0.3447 0.10736 0.063"/>
-  <xacro:property name="body_mass" value="6.5" />
-  <xacro:property name="volume" value="0.005295219" />
+  <xacro:property name="body_mass" value="16.32852408" />
+  <xacro:property name="tail_mass" value="0.59421936" />
   <xacro:property name="model_name" value="Tail_zapolnennie.STL" />
 <!-- Creating reference frame  -->
@@ -25,11 +25,11 @@
         <!--<mesh filename="file://$(find fish)/meshes/${model_name}" scale="${mesh_scale}" />-->
       </geometry>
-      <origin rpy="0.0 0.0 0.0" xyz="0.0 0.0 0.0" />
+      <origin rpy="0.0 0.0 0.0" xyz="0.363 0.103 0.053" />
     </collision>
     <inertial>
-      <origin rpy="0.0 0.0 0.0" xyz="${body_center_gravity}"/>
+      <origin rpy="0.0 0.0 0.0" xyz="0.0 0.0 0.0"/>
       <mass value="${body_mass}"/>
-      <inertia ixx="0.022636377" ixy="0.001191355" ixz="0.0"
-        iyy="0.142422100" iyz="0.0"  izz="0.15464559"/>
+      <inertia ixx="0.77494088896" ixy="0.0" ixz="0.0"
+        iyy="0.07303204514" iyz="0.0"  izz="0.142422100"/>
     </inertial>
   </link>
@@ -54,8 +54,8 @@
     </collision>
     <inertial>
-      <origin rpy="0.0 0.0 0.0" xyz="0.14137 0.0 0.0"/>
-      <mass value="0.687"/>
-      <inertia ixx="0.000273771" ixy="0.0" ixz="0.0"
-        iyy="0.00075492555" iyz="0.0"  izz="0.00102785965"/>
+      <origin rpy="0.0 0.0 0.0" xyz="0.14147 0.0 0.0"/>
+      <mass value="${tail_mass}"/>
+      <inertia ixx="0.00218880737" ixy="0.0" ixz="0.0"
+        iyy="0.00366861219" iyz="0.0"  izz="0.005387317"/>
     </inertial>
   </link>
@@ -93,10 +93,10 @@
     <plugin name="buoyancy" filename="libBuoyancyPlugin.so">
       <link name="body_link">
-        <center_of_volume>0.3447 0.10736 0.0630</center_of_volume>
-        <volume>0.005830207</volume>
+        <!--<center_of_volume></center_of_volume>-->
+        <volume>0.015852936</volume>
       </link>
       <link name="tail_link">
-        <center_of_volume>0.14137 0.12445 0.02142</center_of_volume>
-        <volume>0.000122907</volume>
+        <!--<center_of_volume>0.14137 0.12445 0.02142</center_of_volume>-->
+        <volume>0.000576912</volume>
       </link>
       <fluid_density>1030</fluid_density>

Commit message: Removed moveit dependency and put inertias

File: urdf/fish.urdf.xacro (robot description, xacro)
@@ -22,11 +22,11 @@
     <collision>
       <geometry>
-        <box size="0.726 0.206 0.106"/>
+        <box size="${0.726 - 0.016} 0.206 0.106"/>
         <!--<mesh filename="file://$(find fish)/meshes/${model_name}" scale="${mesh_scale}" />-->
       </geometry>
-      <origin rpy="0.0 0.0 0.0" xyz="0.363 0.103 0.053" />
+      <origin rpy="0.0 0.0 0.0" xyz="0.363 ${0.103 + 0.010} ${0.053 + 0.011}" />
     </collision>
     <inertial>
-      <origin rpy="0.0 0.0 0.0" xyz="0.0 0.0 0.0"/>
+      <origin rpy="0.0 0.0 0.0" xyz="0.363 ${0.103 + 0.010} ${0.053 + 0.011}" />
       <mass value="${body_mass}"/>
       <inertia ixx="0.77494088896" ixy="0.0" ixz="0.0"
@@ -48,5 +48,5 @@
     <collision>
       <geometry>
-        <box size="0.272 0.210 0.0101"/>
+        <box size="${0.272 - 0.022} 0.210 0.0101"/>
         <!--<mesh filename="file://$(find fish)/meshes/Tail.STL" scale="${mesh_scale}" />-->
       </geometry>

Commit message: Fixed inertias

File: urdf/fish.urdf.xacro (robot description, xacro)
@@ -2,6 +2,5 @@
 <robot name="fish" xmlns:xacro="http://www.ros.org/wiki/xacro">
   <xacro:property name="mesh_scale" value="0.001 0.001 0.001" />
-  <xacro:property name="body_center_gravity" value="0.3447 0.10736 0.063"/>
-  <xacro:property name="body_mass" value="16.32852408" />
+  <xacro:property name="body_mass" value="${16.32852408}" />
   <xacro:property name="tail_mass" value="0.59421936" />
   <xacro:property name="model_name" value="Tail_zapolnennie.STL" />
@@ -30,6 +29,6 @@
       <origin rpy="0.0 0.0 0.0" xyz="0.363 ${0.103 + 0.010} ${0.053 + 0.011}" />
       <mass value="${body_mass}"/>
-      <inertia ixx="0.77494088896" ixy="0.0" ixz="0.0"
-        iyy="0.07303204514" iyz="0.0"  izz="0.142422100"/>
+      <inertia ixx="0.07303204514" ixy="0.0" ixz="0.0"
+        iyy="0.7348682585" iyz="0.0"  izz="0.77494088896"/>
     </inertial>
   </link>
@@ -57,5 +56,5 @@
       <mass value="${tail_mass}"/>
       <inertia ixx="0.00218880737" ixy="0.0" ixz="0.0"
-        iyy="0.00366861219" iyz="0.0"  izz="0.005387317"/>
+        iyy="0.00366861219" iyz="0.0"  izz="0.00584731684"/>
     </inertial>
   </link>
@@ -65,5 +64,5 @@
     <origin rpy="0.0 0.0 0.0" xyz="0.71715009 0.1144113 0.06308235"/>
     <axis xyz="0 1 0"/>
-    <limit lower="${-pi/6}" upper="${pi/6}" velocity="${pi/2}" effort="30" />
+    <limit lower="${-pi/6}" upper="${pi/6}" velocity="${pi/2}" effort="100" />
   </joint>
   <!-- CONTROL PLUGIN -->

Commit message: Added cylinder and its' inertias

File: urdf/fish.urdf.xacro (robot description, xacro)
@@ -2,6 +2,6 @@
 <robot name="fish" xmlns:xacro="http://www.ros.org/wiki/xacro">
   <xacro:property name="mesh_scale" value="0.001 0.001 0.001" />
-  <xacro:property name="body_mass" value="${16.32852408}" />
-  <xacro:property name="tail_mass" value="0.59421936" />
+  <xacro:property name="body_mass" value="${23.343741186}" />
+  <xacro:property name="tail_mass" value="${0.6044864}" />
   <xacro:property name="model_name" value="Tail_zapolnennie.STL" />
 <!-- Creating reference frame  -->
@@ -21,14 +21,15 @@
     <collision>
       <geometry>
-        <box size="${0.726 - 0.016} 0.206 0.106"/>
+        <cylinder radius="${0.206 / 2}" length="${0.726 - 0.046}" />
+        <!--<box size="${0.726 - 0.016} 0.206 0.106"/> -->
         <!--<mesh filename="file://$(find fish)/meshes/${model_name}" scale="${mesh_scale}" />-->
       </geometry>
-      <origin rpy="0.0 0.0 0.0" xyz="0.363 ${0.103 + 0.010} ${0.053 + 0.011}" />
+      <origin rpy="0.0 ${pi/2} 0.0" xyz="0.363 ${0.103 + 0.010} ${0.053 + 0.011}" />
     </collision>
     <inertial>
       <origin rpy="0.0 0.0 0.0" xyz="0.363 ${0.103 + 0.010} ${0.053 + 0.011}" />
       <mass value="${body_mass}"/>
-      <inertia ixx="0.07303204514" ixy="0.0" ixz="0.0"
-        iyy="0.7348682585" iyz="0.0"  izz="0.77494088896"/>
+      <inertia ixx="0.123826875" ixy="0.0" ixz="0.0"
+        iyy="0.961425598" iyz="0.0"  izz="0.961425598"/>
     </inertial>
   </link>
@@ -47,5 +48,6 @@
     <collision>
       <geometry>
-        <box size="${0.272 - 0.022} 0.210 0.0101"/>
+        <cylinder radius="${0.272 / 2.0}" length="${0.0101}" />
+        <!--<box size="${0.272 - 0.022} 0.210 0.0101"/> -->
         <!--<mesh filename="file://$(find fish)/meshes/Tail.STL" scale="${mesh_scale}" />-->
       </geometry>
@@ -55,6 +57,6 @@
       <origin rpy="0.0 0.0 0.0" xyz="0.14147 0.0 0.0"/>
       <mass value="${tail_mass}"/>
-      <inertia ixx="0.00218880737" ixy="0.0" ixz="0.0"
-        iyy="0.00366861219" iyz="0.0"  izz="0.00584731684"/>
+      <inertia ixx="0.002800282" ixy="0.0" ixz="0.0"
+        iyy="0.005590287" iyz="0.0"  izz="0.005590287"/>
     </inertial>
   </link>
@@ -93,9 +95,9 @@
       <link name="body_link">
         <!--<center_of_volume></center_of_volume>-->
-        <volume>0.015852936</volume>
+        <volume>0.022663826</volume>
       </link>
       <link name="tail_link">
         <!--<center_of_volume>0.14137 0.12445 0.02142</center_of_volume>-->
-        <volume>0.000576912</volume>
+        <volume>0.00058688</volume>
       </link>
       <fluid_density>1030</fluid_density>

Commit message: WORKS!

File: urdf/fish.urdf.xacro (robot description, xacro)
@@ -43,5 +43,4 @@
         <color rgba="0.2 1.0 0.2 1.0"/>
       </material>
-    <!--xyz="0.70705 -0.01004 0.04165"-->
       <origin rpy="0.0 0.0 0.0" xyz="-0.0101009 -0.1244513 -0.02143235"/>
     </visual>
@@ -49,6 +48,4 @@
       <geometry>
         <cylinder radius="${0.272 / 2.0}" length="${0.0101}" />
-        <!--<box size="${0.272 - 0.022} 0.210 0.0101"/> -->
-        <!--<mesh filename="file://$(find fish)/meshes/Tail.STL" scale="${mesh_scale}" />-->
       </geometry>
       <origin rpy="0.0 0.0 0.0" xyz="0.14147 0.0 0.0"/>
@@ -58,5 +55,5 @@
       <mass value="${tail_mass}"/>
       <inertia ixx="0.002800282" ixy="0.0" ixz="0.0"
-        iyy="0.005590287" iyz="0.0"  izz="0.005590287"/>
+        iyy="0.002800282" iyz="0.0"  izz="0.005590287"/>
     </inertial>
   </link>
@@ -67,5 +64,5 @@
     <axis xyz="0 1 0"/>
     <limit lower="${-pi/6}" upper="${pi/6}" velocity="${pi/2}" effort="100" />
-  </joint>
+  </joint>-->
   <!-- CONTROL PLUGIN -->
 	<joint name="world_joint" type="floating">
@@ -94,9 +91,9 @@
     <plugin name="buoyancy" filename="libBuoyancyPlugin.so">
       <link name="body_link">
-        <!--<center_of_volume></center_of_volume>-->
+        <center_of_volume>0.363 0.113 0.064</center_of_volume>
         <volume>0.022663826</volume>
       </link>
       <link name="tail_link">
-        <!--<center_of_volume>0.14137 0.12445 0.02142</center_of_volume>-->
+        <center_of_volume>0.14147 0.0 0.0</center_of_volume>
         <volume>0.00058688</volume>
       </link>

Commit message: Tuned all the parameters

File: urdf/fish.urdf.xacro (robot description, xacro)
@@ -52,5 +52,5 @@
     </collision>
     <inertial>
-      <origin rpy="0.0 0.0 0.0" xyz="0.14147 0.0 0.0"/>
+      <origin rpy="0.0 0.0 0.0" xyz="0.14147 -0.0005 0.0"/>
       <mass value="${tail_mass}"/>
       <inertia ixx="0.002800282" ixy="0.0" ixz="0.0"
@@ -63,6 +63,6 @@
     <origin rpy="0.0 0.0 0.0" xyz="0.71715009 0.1144113 0.06308235"/>
     <axis xyz="0 1 0"/>
-    <limit lower="${-pi/6}" upper="${pi/6}" velocity="${pi/2}" effort="100" />
-  </joint>-->
+    <limit lower="${-pi/2}" upper="${pi/2}" velocity="${pi}" effort="10000" />
+  </joint>
   <!-- CONTROL PLUGIN -->
 	<joint name="world_joint" type="floating">
@@ -103,14 +103,15 @@
       <link_name>tail_link</link_name>
       <air_density>1030</air_density>
-      <cla>0.2969</cla>
-      <cla_stall>-0.1044</cla_stall>
-      <cda>0</cda>
-      <cda_stall>0.1044</cda_stall>
-      <alpha_stall>0.3368</alpha_stall>
-      <a0>0</a0>
-      <area>0.041820095</area>
-      <upward>-0.330514 0.943801 0</upward>
-      <forward>0.943801  0.330514 0</forward>
-      <cp>0.14137 0.12445 0.02142</cp>
+      <a0>0.08727</a0>
+      <alpha_stall>${pi/6}</alpha_stall>
+      <cla>0.08727</cla>
+      <cla_stall>${pi/6}</cla_stall>
+      <cda>0.0</cda>
+      <cda_stall>0.0</cda_stall>
+      <area>0.1248444</area>
+      <!--<area>0.058106898</area>-->
+      <upward>0.0 0.0 1.0</upward>
+      <forward>-1.0 0.0 0.0</forward>
+      <cp>0.14147 -0.0007 0.0</cp>
     </plugin>
   </gazebo>

Commit message: New fish works

File: urdf/fish.urdf.xacro (robot description, xacro)
@@ -4,5 +4,6 @@
   <xacro:property name="body_mass" value="${23.343741186}" />
   <xacro:property name="tail_mass" value="${0.6044864}" />
-  <xacro:property name="model_name" value="Tail_zapolnennie.STL" />
+  <xacro:property name="model_name" value="Rework/Body_only.STL" />
+  <xacro:property name="tail_name" value="Rework/hvost.STL" />
 <!-- Creating reference frame  -->
   <link name="world" />
@@ -17,5 +18,5 @@
         <color rgba="0.2 1.0 0.2 1.0"/>
       </material>
-      <origin rpy="0.0 0.0 0.0" xyz="0.0 0.0 0.0" />
+      <origin rpy="0.0 ${-pi/2} 0.0" xyz="0.740 -0.025 -0.07" />
     </visual>
     <collision>
@@ -38,5 +39,5 @@
     <visual>
       <geometry>
-        <mesh filename="file://$(find fish)/meshes/Tail.STL" scale="${mesh_scale}"/>
+        <mesh filename="file://$(find fish)/meshes/${tail_name}" scale="${mesh_scale}"/>
       </geometry>
       <material name="Green">
